Commit message: still i couldn't realize depth measurement

File: ros2_ws/src/gazebo_turtlebot3/urdf/turtlebot3_waffle_pi_close.urdf (robot description, URDF)
Before this commit: robot turtlebot3_waffle_pi, 11 links, 10 joints
Links:
- added link camera_depth_optical_frame
- added link realsense_depth_frame
Joints:
- added joint camera_depth_optical_joint: type fixed, parent realsense_depth_frame, child camera_depth_optical_frame, origin xyz=0 0 0 rpy=-1.57 0 -1.57
- added joint realsense_depth_joint: type fixed, parent camera_link, child realsense_depth_frame, origin xyz=0.003 0.011 0.009 rpy=0 0 0
